File: pcb/SoundBoard.kicad_pcb (KiCad board)
At the start: 2 copper layers, 50 x 85 mm, 13 parts, among them J1 Micro SD Card Adapter, J2 Barrel_Jack_Switch, J3 Conn_01x04_Socket, U1 ESP32-DEVKIT-V1, U2_L1 DEV14809, U2_R1 DEV14809

Commit message: Improved PCBs (REV2.0)
Parts:
- C1, C2, C3: value C_Polarized -> 470uF
- D1: value D_Schottky -> 1N5822; footprint Diode_SMD:D_SOD-123 -> Diode_SMD:D_SMA_Handsoldering
Other:
- board text added: "REV2.0 2024/11 by foorschtbar"
- board text removed: "REV1.0 2024/10 by foorschtbar"
Changed lines of the file:
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@@
 		(pad_to_mask_clearance 0)
 		(allow_soldermask_bridges_in_footprints no)
-		(grid_origin 78.835 108.15)
+		(grid_origin 183.985 58.21)
 		(pcbplotparams
 			(layerselection 0x00010fc_ffffffff)
@@
 			)
 		)
-		(property "Value" "C_Polarized"
+		(property "Value" "470uF"
 			(at 0 4.35 0)
 			(layer "F.Fab")
@@
 			)
 		)
-		(property "Value" "C_Polarized"
+		(property "Value" "470uF"
 			(at 0 4.35 0)
 			(layer "F.Fab")
@@
 			)
 		)
-		(property "Value" "C_Polarized"
+		(property "Value" "470uF"
 			(at 0 4.35 0)
 			(layer "F.Fab")
@@
 		)
 	)
-	(footprint "Diode_SMD:D_SOD-123"
+	(footprint "Diode_SMD:D_SMA_Handsoldering"
 		(layer "F.Cu")
 		(at 173.485 75.21)
-		(descr "SOD-123")
-		(tags "SOD-123")
+		(descr "Diode SMA (DO-214AC) Handsoldering")
+		(tags "Diode SMA (DO-214AC) Handsoldering")
 		(property "Reference" "D1"
-			(at 3.4 0 0)
+			(at 5.6 -0.06 0)
 			(layer "F.SilkS")
 			(effects
@@
 			)
 		)
-		(property "Value" "D_Schottky"
-			(at 0 2.1 0)
+		(property "Value" "1N5822"
+			(at 0 2.6 0)
 			(layer "F.Fab")
-			(hide yes)
 			(effects
 				(font
@@
 			)
 		)
-		(property "Footprint" "Diode_SMD:D_SOD-123"
+		(property "Footprint" "Diode_SMD:D_SMA_Handsoldering"
 			(at 0 0 0)
 			(unlocked yes)
@@
 		(attr smd)
 		(fp_line
-			(start -2.36 -1)
-			(end -2.36 1)
+			(start -4.51 -1.65)
+			(end -4.51 1.65)
 			(stroke
 				(width 0.12)
@@
 		)
 		(fp_line
-			(start -2.36 -1)
-			(end 1.65 -1)
+			(start -4.51 -1.65)
+			(end 2.5 -1.65)
 			(stroke
 				(width 0.12)
@@
 		)
 		(fp_line
-			(start -2.36 1)
-			(end 1.65 1)
+			(start -4.51 1.65)
+			(end 2.5 1.65)
 			(stroke
 				(width 0.12)
@@
 		)
 		(fp_line
-			(start -2.35 -1.15)
-			(end -2.35 1.15)
+			(start -4.5 -1.75)
+			(end 4.5 -1.75)
 			(stroke
 				(width 0.05)
@@
 		)
 		(fp_line
-			(start -2.35 -1.15)
-			(end 2.35 -1.15)
+			(start -4.5 1.75)
+			(end -4.5 -1.75)
 			(stroke
 				(width 0.05)
@@
 		)
 		(fp_line
-			(start 2.35 -1.15)
-			(end 2.35 1.15)
+			(start 4.5 -1.75)
+			(end 4.5 1.75)
 			(stroke
 				(width 0.05)
@@
 		)
 		(fp_line
-			(start 2.35 1.15)
-			(end -2.35 1.15)
+			(start 4.5 1.75)
+			(end -4.5 1.75)
 			(stroke
 				(width 0.05)
@@
 		)
 		(fp_line
-			(start -1.4 -0.9)
-			(end 1.4 -0.9)
-			(stroke
-				(width 0.1)
-				(type solid)
-			)
-			(layer "F.Fab")
-		)
-		(fp_line
-			(start -1.4 0.9)
-			(end -1.4 -0.9)
+			(start -2.3 1.5)
+			(end -2.3 -1.5)
 			(stroke
 				(width 0.1)
@@
 		)
 		(fp_line
-			(start -0.75 0)
-			(end -0.35 0)
+			(start -0.64944 -0.79908)
+			(end -0.64944 0.80112)
 			(stroke
 				(width 0.1)
@@
 		)
 		(fp_line
-			(start -0.35 0)
-			(end -0.35 -0.55)
+			(start -0.64944 0.00102)
+			(end -1.55114 0.00102)
 			(stroke
 				(width 0.1)
@@
 		)
 		(fp_line
-			(start -0.35 0)
-			(end -0.35 0.55)
+			(start -0.64944 0.00102)
+			(end 0.50118 -0.79908)
 			(stroke
 				(width 0.1)
@@
 		)
 		(fp_line
-			(start -0.35 0)
-			(end 0.25 -0.4)
+			(start -0.64944 0.00102)
+			(end 0.50118 0.75032)
 			(stroke
 				(width 0.1)
@@
 		)
 		(fp_line
-			(start 0.25 -0.4)
-			(end 0.25 0.4)
+			(start 0.50118 0.00102)
+			(end 1.4994 0.00102)
 			(stroke
 				(width 0.1)
@@
 		)
 		(fp_line
-			(start 0.25 0)
-			(end 0.75 0)
+			(start 0.50118 0.75032)
+			(end 0.50118 -0.79908)
 			(stroke
 				(width 0.1)
@@
 		)
 		(fp_line
-			(start 0.25 0.4)
-			(end -0.35 0)
+			(start 2.3 -1.5)
+			(end -2.3 -1.5)
 			(stroke
 				(width 0.1)
@@
 		)
 		(fp_line
-			(start 1.4 -0.9)
-			(end 1.4 0.9)
+			(start 2.3 -1.5)
+			(end 2.3 1.5)
 			(stroke
 				(width 0.1)
@@
 		)
 		(fp_line
-			(start 1.4 0.9)
-			(end -1.4 0.9)
+			(start 2.3 1.5)
+			(end -2.3 1.5)
 			(stroke
 				(width 0.1)
@@
 		)
 		(fp_text user "${REFERENCE}"
-			(at 0 -2 0)
+			(at 0 -2.5 0)
 			(layer "F.Fab")
-			(hide yes)
 			(effects
 				(font
@@
 		)
 		(pad "1" smd roundrect
-			(at -1.65 0)
-			(size 0.9 1.2)
+			(at -2.5 0)
+			(size 3.5 1.8)
 			(layers "F.Cu" "F.Paste" "F.Mask")
-			(roundrect_rratio 0.25)
+			(roundrect_rratio 0.1388888889)
 			(net 3 "/VIN")
 			(pinfunction "K")
@@
 		)
 		(pad "2" smd roundrect
-			(at 1.65 0)
-			(size 0.9 1.2)
+			(at 2.5 0)
+			(size 3.5 1.8)
 			(layers "F.Cu" "F.Paste" "F.Mask")
-			(roundrect_rratio 0.25)
+			(roundrect_rratio 0.1388888889)
 			(net 1 "+5V")
 			(pinfunction "A")
 			(pintype "passive")
 		)
-		(model "${KICAD8_3DMODEL_DIR}/Diode_SMD.3dshapes/D_SOD-123.wrl"
+		(model "${KICAD8_3DMODEL_DIR}/Diode_SMD.3dshapes/D_SMA.wrl"
 			(offset
 				(xyz 0 0 0)
@@
 	)
 	(gr_circle
-		(center 151.245 135.554999)
-		(end 150.245 135.554999)
+		(center 156.425 135.245001)
+		(end 157.425 135.245001)
 		(stroke
 			(width 0.2)
@@
 	)
 	(gr_line
-		(start 156.925 135.429999)
-		(end 155.725 135.429999)
+		(start 150.745 135.370001)
+		(end 151.945 135.370001)
 		(stroke
 			(width 0.2)
@@
 	)
 	(gr_circle
-		(center 166.605 135.429999)
-		(end 165.605 135.429999)
+		(center 161.565 135.370001)
+		(end 162.565 135.370001)
 		(stroke
 			(width 0.2)
@@
 	)
 	(gr_line
-		(start 162.125 135.554999)
-		(end 160.925 135.554999)
+		(start 166.045 135.245001)
+		(end 167.245 135.245001)
 		(stroke
 			(width 0.2)
@@
 	)
 	(gr_circle
-		(center 161.525 135.554999)
-		(end 160.525 135.554999)
+		(center 166.645 135.245001)
+		(end 167.645 135.245001)
 		(stroke
 			(width 0.2)
@@
 	)
 	(gr_line
-		(start 166.605 134.829999)
-		(end 166.605 136.029999)
+		(start 161.565 135.970001)
+		(end 161.565 134.770001)
 		(stroke
 			(width 0.2)
@@
 	)
 	(gr_circle
-		(center 156.325 135.429999)
-		(end 155.325 135.429999)
+		(center 151.345 135.370001)
+		(end 152.345 135.370001)
 		(stroke
 			(width 0.2)
@@
 	)
 	(gr_line
-		(start 167.205 135.429999)
-		(end 166.005 135.429999)
+		(start 160.965 135.370001)
+		(end 162.165 135.370001)
 		(stroke
 			(width 0.2)
@@
 	)
 	(gr_line
-		(start 156.325 134.829999)
-		(end 156.325 136.029999)
+		(start 151.345 135.970001)
+		(end 151.345 134.770001)
 		(stroke
 			(width 0.2)
@@
 	)
 	(gr_line
-		(start 151.845 135.554999)
-		(end 150.645 135.554999)
+		(start 155.825 135.245001)
+		(end 157.025 135.245001)
 		(stroke
 			(width 0.2)
@@
 	)
 	(gr_rect
-		(start 120.535 75.305)
-		(end 123.535 160.305)
+		(start 180.985 58.21)
+		(end 183.985 143.21)
 		(stroke
 			(width 0.1)
@@
 		)
 		(fill solid)
-		(layer "F.Mask")
+		(layer "B.Mask")
 	)
 	(gr_rect
-		(start 120.535 75.305)
-		(end 123.535 160.305)
+		(start 133.985 58.21)
+		(end 136.985 143.21)
+		(stroke
+			(width 0.1)
+			(type default)
+		)
+		(fill solid)
+		(layer "B.Mask")
+	)
+	(gr_rect
+		(start 180.985 58.21)
+		(end 183.985 143.21)
 		(stroke
 			(width 0.1)
@@
 	)
 	(gr_rect
-		(start 73.535 75.305)
-		(end 76.535 160.305)
+		(start 133.985 58.21)
+		(end 136.985 143.21)
 		(stroke
 			(width 0.1)
@@
 	)
 	(gr_text "RIGHT"
-		(at 164.065 135.305 90)
+		(at 164.105 135.495 -90)
 		(layer "B.SilkS")
 		(effects
@@
 	)
 	(gr_text "LEFT"
-		(at 153.785 135.305 90)
+		(at 153.885 135.495 -90)
 		(layer "B.SilkS")
 		(effects
@@
 		)
 	)
-	(gr_text "REV1.0 2024/10\nby foorschtbar\n"
+	(gr_text "REV2.0 2024/11\nby foorschtbar\n"
 		(at 158.785 123.305 0)
 		(layer "B.SilkS")
@@
 		)
 	)
-	(gr_text "REV1.0 2024/10\nby foorschtbar\n"
+	(gr_text "REV2.0 2024/11\nby foorschtbar\n"
 		(at 176.285 97.555 90)
 		(layer "F.SilkS")
@@
 		(layer "User.1")
 		(pts
-			(xy 73.535 160.305) (xy 73.535 75.305)
+			(xy 133.985 143.21) (xy 133.985 58.21)
 		)
 		(height -9)
 		(gr_text "85.0000 mm"
-			(at 63.385 117.805 90)
+			(at 123.835 100.71 90)
 			(layer "User.1")
 			(effects
@@
 		(layer "User.1")
 		(pts
-			(xy 73.535 160.305) (xy 123.535 160.305)
+			(xy 133.985 143.21) (xy 183.985 143.21)
 		)
 		(height 12.965)
 		(gr_text "50.0000 mm"
-			(at 98.535 172.12 0)
+			(at 158.985 155.025 0)
 			(layer "User.1")
 			(effects

Commit message: PCB Rev 2.1
Connections:
- D1 pad 1: /VIN -> VIN
- J1 pad 2: +5V -> VIN
- LED1 pad 2: +5V -> VIN
- U1 pad 30: /VIN -> VIN
Routing:
- net VIN: track 0.00 -> 56.8 mm
- net +5V: track 176.9 -> 138.1 mm
- net /VIN: track 9.92 -> 0.00 mm
Other:
- board text added: "REV2.1 2024/12 by foorschtbar"
- board text removed: "REV2.0 2024/11 by foorschtbar"
Changed lines of the file:
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@@
 		(pad_to_mask_clearance 0)
 		(allow_soldermask_bridges_in_footprints no)
-		(grid_origin 183.985 58.21)
+		(grid_origin 139.285 103.755)
 		(pcbplotparams
 			(layerselection 0x00010fc_ffffffff)
@@
 	(net 1 "+5V")
 	(net 2 "GND")
-	(net 3 "/VIN")
+	(net 3 "VIN")
 	(net 4 "Net-(J3-Pin_2)")
 	(net 5 "Net-(J3-Pin_1)")
@@
 			(layers "*.Cu" "*.Mask")
 			(remove_unused_layers no)
-			(net 3 "/VIN")
+			(net 3 "VIN")
 			(pinfunction "VIN")
 			(pintype "input")
@@
 			(size 0.7 1.2)
 			(layers "F.Cu" "F.Paste" "F.Mask")
-			(net 1 "+5V")
+			(net 3 "VIN")
 			(pinfunction "VDD")
 			(pintype "passive")
@@
 			(layers "F.Cu" "F.Paste" "F.Mask")
 			(roundrect_rratio 0.1388888889)
-			(net 3 "/VIN")
+			(net 3 "VIN")
 			(pinfunction "K")
 			(pintype "passive")
@@
 			(layers "*.Cu" "*.Mask")
 			(remove_unused_layers no)
-			(net 1 "+5V")
+			(net 3 "VIN")
 			(pinfunction "VCC")
 			(pintype "power_in")
@@
 		)
 	)
+	(gr_poly
+		(pts
+			(xy 166.935 104.505) (xy 166.935 103.005) (xy 165.935 103.755)
+		)
+		(stroke
+			(width 0.1)
+			(type solid)
+		)
+		(fill solid)
+		(layer "B.SilkS")
+	)
+	(gr_poly
+		(pts
+			(xy 136.985 85.225) (xy 136.985 86.725) (xy 137.985 85.975)
+		)
+		(stroke
+			(width 0.1)
+			(type solid)
+		)
+		(fill solid)
+		(layer "B.SilkS")
+	)
 	(gr_circle
 		(center 156.425 135.245001)
@@
 		(layer "B.SilkS")
 	)
+	(gr_poly
+		(pts
+			(xy 136.985 103.005) (xy 136.985 104.505) (xy 137.985 103.755)
+		)
+		(stroke
+			(width 0.1)
+			(type solid)
+		)
+		(fill solid)
+		(layer "B.SilkS")
+	)
 	(gr_circle
 		(center 161.565 135.370001)
@@
 		(layer "B.SilkS")
 	)
+	(gr_poly
+		(pts
+			(xy 166.935 81.645) (xy 166.935 80.145) (xy 165.935 80.895)
+		)
+		(stroke
+			(width 0.1)
+			(type solid)
+		)
+		(fill solid)
+		(layer "B.SilkS")
+	)
+	(gr_poly
+		(pts
+			(xy 166.935 86.725) (xy 166.935 85.225) (xy 165.935 85.975)
+		)
+		(stroke
+			(width 0.1)
+			(type solid)
+		)
+		(fill solid)
+		(layer "B.SilkS")
+	)
+	(gr_poly
+		(pts
+			(xy 136.985 69.96) (xy 136.985 71.46) (xy 137.985 70.71)
+		)
+		(stroke
+			(width 0.1)
+			(type solid)
+		)
+		(fill solid)
+		(layer "B.SilkS")
+	)
+	(gr_poly
+		(pts
+			(xy 166.935 68.945) (xy 166.935 67.445) (xy 165.935 68.195)
+		)
+		(stroke
+			(width 0.1)
+			(type solid)
+		)
+		(fill solid)
+		(layer "B.SilkS")
+	)
 	(gr_line
 		(start 166.045 135.245001)
@@
 		(layer "B.SilkS")
 	)
+	(gr_poly
+		(pts
+			(xy 166.935 74.025) (xy 166.935 72.525) (xy 165.935 73.275)
+		)
+		(stroke
+			(width 0.1)
+			(type solid)
+		)
+		(fill solid)
+		(layer "B.SilkS")
+	)
+	(gr_poly
+		(pts
+			(xy 166.935 84.185) (xy 166.935 82.685) (xy 165.935 83.435)
+		)
+		(stroke
+			(width 0.1)
+			(type solid)
+		)
+		(fill solid)
+		(layer "B.SilkS")
+	)
 	(gr_circle
 		(center 166.645 135.245001)
@@
 		(layer "B.SilkS")
 	)
+	(gr_poly
+		(pts
+			(xy 166.935 71.485) (xy 166.935 69.985) (xy 165.935 70.735)
+		)
+		(stroke
+			(width 0.1)
+			(type solid)
+		)
+		(fill solid)
+		(layer "B.SilkS")
+	)
 	(gr_line
 		(start 161.565 135.970001)
@@
 		(layer "B.SilkS")
 	)
+	(gr_poly
+		(pts
+			(xy 136.985 87.765) (xy 136.985 89.265) (xy 137.985 88.515)
+		)
+		(stroke
+			(width 0.1)
+			(type solid)
+		)
+		(fill solid)
+		(layer "B.SilkS")
+	)
 	(gr_line
 		(start 160.965 135.370001)
@@
 		(layer "B.SilkS")
 	)
+	(gr_poly
+		(pts
+			(xy 136.985 90.305) (xy 136.985 91.805) (xy 137.985 91.055)
+		)
+		(stroke
+			(width 0.1)
+			(type solid)
+		)
+		(fill solid)
+		(layer "B.SilkS")
+	)
 	(gr_line
 		(start 167.385 131.775)
@@
 		)
 	)
-	(gr_text "REV2.0 2024/11\nby foorschtbar\n"
+	(gr_text "REV2.1 2024/12\nby foorschtbar\n"
 		(at 158.785 123.305 0)
 		(layer "B.SilkS")
@@
 		)
 	)
-	(gr_text "REV2.0 2024/11\nby foorschtbar\n"
+	(gr_text "REV2.1 2024/12\nby foorschtbar\n"
 		(at 176.285 97.555 90)
 		(layer "F.SilkS")
@@
 	)
 	(segment
-		(start 155.795 96.4)
-		(end 155.795 110.175)
-		(width 1)
-		(layer "F.Cu")
-		(net 1)
-	)
-	(segment
 		(start 173.485 70.51)
 		(end 173.485 68.51)
@@
 	)
 	(segment
-		(start 152.435 60.705)
-		(end 152.435 59.91)
-		(width 0.25)
-		(layer "F.Cu")
-		(net 1)
-	)
-	(segment
 		(start 173.485 78.8875)
 		(end 170.9475 81.425)
@@
 	)
 	(segment
-		(start 168.03 63.055)
-		(end 154.785 63.055)
-		(width 0.25)
-		(layer "F.Cu")
-		(net 1)
-	)
-	(segment
-		(start 173.485 68.51)
-		(end 168.03 63.055)
-		(width 0.25)
-		(layer "F.Cu")
-		(net 1)
-	)
-	(segment
 		(start 155.795 110.175)
 		(end 145.735 110.175)
@@
 	)
 	(segment
-		(start 154.785 63.055)
-		(end 152.435 60.705)
-		(width 0.25)
-		(layer "F.Cu")
-		(net 1)
-	)
-	(segment
 		(start 173.985 136.6725)
 		(end 172.4475 138.21)
@@
 	)
 	(segment
+		(start 155.795 96.4)
+		(end 155.795 68.265)
+		(width 0.25)
+		(layer "F.Cu")
+		(net 3)
+	)
+	(segment
 		(start 171.7 75.21)
 		(end 164.685 68.195)
@@
 		(layer "F.Cu")
 		(net 3)
+	)
+	(segment
+		(start 164.685 68.195)
+		(end 155.725 68.195)
+		(width 0.25)
+		(layer "F.Cu")
+		(net 3)
+	)
+	(segment
+		(start 152.435 64.905)
+		(end 152.435 59.91)
+		(width 0.25)
+		(layer "F.Cu")
+		(net 3)
+	)
+	(segment
+		(start 155.795 68.265)
+		(end 155.725 68.195)
+		(width 0.25)
+		(layer "F.Cu")
+		(net 3)
+	)
+	(segment
+		(start 155.725 68.195)
+		(end 152.435 64.905)
+		(width 0.25)
+		(layer "F.Cu")
+		(net 3)
