File: pcb/SoundBoard.kicad_sch (KiCad schematic)
At the start: 11 parts, among them J1 Micro SD Card Adapter, J2 Barrel_Jack, J3 Conn_01x02_Socket, J4 Conn_01x02_Socket, U1 ESP32-DEVKIT-V1, U2_L DEV14809, U2_R DEV14809

Commit message: Fixed left channel
Connections:
- net +5V: now also U2_L.J2_5 (~{SD})
- no-connect marks 21 -> 20
Changed lines of the file:
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@@
-	)
-	(no_connect
-		(at 191.77 60.96)
 	)
 	(no_connect
@@
 					(unit 1)
 				)
+			)
+		)
+	)
+	(symbol
+		(lib_id "power:+5V")
+		(at 191.77 60.96 90)
+		(unit 1)
+		(exclude_from_sim no)
+		(in_bom yes)
+		(on_board yes)
+		(dnp no)
+		(fields_autoplaced yes)
+		(property "Reference" "#PWR016"
+			(at 195.58 60.96 0)
+			(effects
+				(font
+					(size 1.27 1.27)
+				)
+				(hide yes)
+			)
+		)
+		(property "Value" "+5V"
+			(at 187.96 60.9599 90)
+			(effects
+				(font
+					(size 1.27 1.27)
+				)
+				(justify left)
+			)
+		)
+		(property "Footprint" ""
+			(at 191.77 60.96 0)
+			(effects
+				(font
+					(size 1.27 1.27)
+				)
+				(hide yes)
+			)
+		)
+		(property "Datasheet" ""
+			(at 191.77 60.96 0)
+			(effects
+				(font
+					(size 1.27 1.27)
+				)
+				(hide yes)
+			)
+		)
+		(property "Description" "Power symbol creates a global label with name \"+5V\""
+			(at 191.77 60.96 0)
+			(effects
+				(font
+					(size 1.27 1.27)
+				)
+				(hide yes)
+			)
+		)
+		(pin "1"
+		)
+		(instances
+			(project "SoundBoard"
+				(path "/a11f05dd-5082-4e0a-aca6-ddee1418cddd"
+					(reference "#PWR016")
+					(unit 1)
+				)

Commit message: Finished PCB Layout
Parts:
- removed J3: Conn_01x02_Socket, symbol Connector:Conn_01x02_Socket
- added C3: C_Polarized, Capacitor_SMD:C_Elec_6.3x7.7, symbol Device:C_Polarized
- added D1: D_Schottky, Diode_SMD:D_SOD-123, symbol Device:D_Schottky
- C1, C2: footprint (none) -> Capacitor_SMD:C_Elec_6.3x7.7
- J1: footprint (none) -> SDCardAdapter:SDCardAdapter
- J2: value Barrel_Jack -> Barrel_Jack_Switch; footprint (none) -> Connector_BarrelJack:BarrelJack_Horizontal; symbol Connector:Barrel_Jack -> Connector:Barrel_Jack_Switch
- J3: renamed from J4; value Conn_01x02_Socket -> Conn_01x04_Socket; footprint (none) -> TerminalBlock_Phoenix:TerminalBlock_Phoenix_MKDS-1,5-4-5.08_1x04_P5.08mm_Horizontal; symbol Connector:Conn_01x02_Socket -> Connector:Conn_01x04_Socket
- LED1: footprint SK6812SIDE -> SK6812SIDE:SK6812SIDE
- R1: footprint (none) -> Resistor_SMD:R_0805_2012Metric_Pad1.20x1.40mm_HandSolder
- U1: footprint ESP32-DEVKIT-V1:MODULE_ESP32_DEVKIT_V1 -> ESP32-DEVKIT-V1:ESP32_DEVKIT_V1
- U2_L1: renamed from U2_L; footprint DEV14809:MODULE_DEV14809 -> MAX98357A:MAX98357A
- U2_R1: renamed from U2_R; footprint DEV14809:MODULE_DEV14809 -> MAX98357A:MAX98357A
Connections:
- net +5V: now also C3.1, D1.2 (A); no longer U1.30 (VIN)
- net GND: now also C3.2
- net at J3.1 (Pin_1): now also U2_L1.J1_1 (OUT+); no longer U2_R1.J1_1 (OUT+)
- net at J3.2 (Pin_2): now also U2_L1.J1_2 (OUT-); no longer U2_R1.J1_2 (OUT-)
- new net: J3.3 (Pin_3), U2_R1.J1_1 (OUT+)
- new net: J3.4 (Pin_4), U2_R1.J1_2 (OUT-)
- new net VIN: D1.1 (K), U1.30 (VIN)
- no-connect marks 20 -> 21

Commit message: Improved PCBs (REV2.0)
Parts:
- C1, C2, C3: value C_Polarized -> 470uF
- D1: value D_Schottky -> 1N5822; footprint Diode_SMD:D_SOD-123 -> Diode_SMD:D_SMA_Handsoldering
Changed lines of the file:
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@@
 			)
 		)
-		(property "Value" "C_Polarized"
+		(property "Value" "470uF"
 			(at 241.3 68.9609 0)
 			(effects
@@
 			)
 		)
-		(property "Value" "D_Schottky"
+		(property "Value" "1N5822"
 			(at 99.3775 69.85 0)
 			(effects
@@
 			)
 		)
-		(property "Footprint" "Diode_SMD:D_SOD-123"
+		(property "Footprint" "Diode_SMD:D_SMA_Handsoldering"
 			(at 99.06 73.66 0)
 			(effects
@@
 			)
 		)
-		(property "Value" "C_Polarized"
+		(property "Value" "470uF"
 			(at 241.3 114.6809 0)
 			(effects
@@
 			)
 		)
-		(property "Value" "C_Polarized"
+		(property "Value" "470uF"
 			(at 113.03 34.6709 0)
 			(effects

Commit message: PCB Rev 2.1
Connections:
- net +5V: no longer J1.2 (VCC), LED1.2 (VDD)
- net VIN: now also J1.2 (VCC), LED1.2 (VDD)
Changed lines of the file:
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@@
+		)
+	)
+	(global_label "VIN"
+		(shape input)
+		(at 48.26 99.06 90)
+		(fields_autoplaced yes)
+		(effects
+			(font
+				(size 1.27 1.27)
+			)
+			(justify left)
+		)
+		(property "Intersheetrefs" "${INTERSHEET_REFS}"
+			(at 48.26 93.0509 90)
+			(effects
+				(font
+					(size 1.27 1.27)
+				)
+				(justify left)
+				(hide yes)
+			)
 		)
 	)
@@
 				)
 				(justify right)
+				(hide yes)
+			)
+		)
+	)
+	(global_label "VIN"
+		(shape input)
+		(at 48.26 64.77 90)
+		(fields_autoplaced yes)
+		(effects
+			(font
+				(size 1.27 1.27)
+			)
+			(justify left)
+		)
+		(property "Intersheetrefs" "${INTERSHEET_REFS}"
+			(at 48.26 58.7609 90)
+			(effects
+				(font
+					(size 1.27 1.27)
+				)
+				(justify left)
 				(hide yes)
 			)
@@
 	)
 	(symbol
-		(lib_id "power:+5V")
-		(at 48.26 99.06 0)
-		(unit 1)
-		(exclude_from_sim no)
-		(in_bom yes)
-		(on_board yes)
-		(dnp no)
-		(fields_autoplaced yes)
-		(property "Reference" "#PWR014"
-			(at 48.26 102.87 0)
-			(effects
-				(font
-					(size 1.27 1.27)
-				)
-				(hide yes)
-			)
-		)
-		(property "Value" "+5V"
-			(at 48.26 93.98 0)
-			(effects
-				(font
-					(size 1.27 1.27)
-				)
-			)
-		)
-		(property "Footprint" ""
-			(at 48.26 99.06 0)
-			(effects
-				(font
-					(size 1.27 1.27)
-				)
-				(hide yes)
-			)
-		)
-		(property "Datasheet" ""
-			(at 48.26 99.06 0)
-			(effects
-				(font
-					(size 1.27 1.27)
-				)
-				(hide yes)
-			)
-		)
-		(property "Description" "Power symbol creates a global label with name \"+5V\""
-			(at 48.26 99.06 0)
-			(effects
-				(font
-					(size 1.27 1.27)
-				)
-				(hide yes)
-			)
-		)
-		(pin "1"
-		)
-		(instances
-			(project "SoundBoard"
-				(path "/a11f05dd-5082-4e0a-aca6-ddee1418cddd"
-					(reference "#PWR014")
-					(unit 1)
-				)
-			)
-		)
-	)
-	(symbol
 		(lib_id "ESP32-DEVKIT-V1:ESP32-DEVKIT-V1")
 		(at 125.73 99.06 0)
@@
 					(unit 1)
 				)
-			)
-		)
-	)
-	(symbol
-		(lib_id "power:+5V")
-		(at 48.26 64.77 0)
-		(unit 1)
-		(exclude_from_sim no)
-		(in_bom yes)
-		(on_board yes)
-		(dnp no)
-		(fields_autoplaced yes)
-		(property "Reference" "#PWR013"
-			(at 48.26 68.58 0)
-			(effects
-				(font
-					(size 1.27 1.27)
-				)
-				(hide yes)
-			)
-		)
-		(property "Value" "+5V"
-			(at 48.26 59.69 0)
-			(effects
-				(font
-					(size 1.27 1.27)
-				)
-			)
-		)
-		(property "Footprint" ""
-			(at 48.26 64.77 0)
-			(effects
-				(font
-					(size 1.27 1.27)
-				)
-				(hide yes)
-			)
-		)
-		(property "Datasheet" ""
-			(at 48.26 64.77 0)
-			(effects
-				(font
-					(size 1.27 1.27)
-				)
-				(hide yes)
-			)
-		)
-		(property "Description" "Power symbol creates a global label with name \"+5V\""
-			(at 48.26 64.77 0)
-			(effects
-				(font
-					(size 1.27 1.27)
-				)
-				(hide yes)
-			)
-		)
-		(pin "1"
-		)
-		(instances
-			(project "SoundBoard"
-				(path "/a11f05dd-5082-4e0a-aca6-ddee1418cddd"
-					(reference "#PWR013")
-					(unit 1)
-				)
